File: EagleFiles/cherrymx1.brd (EAGLE design)
At the start: 109.2 x 25.4 mm, 23 parts, among them Q1 MMBT2222A, Y1 16MHz

Commit message: Add a bunch more switches!
Parts:
- added R10, R11, R12, R13, R14, R15, R16, R17, R18, R19, R20, R21, R22, R23, R8, R9: 330, adafruit:R0603
- added S10, S11, S12, S13, S14, S15, S16, S17, S18, S19, S20, S5, S6, S7, S8, S9: CHERRY-MX-LED, SparkFun-Electromechanical2:CHERRY-MX-LED
- moved S4 57.2 mm to (96.5, 69.8)
- moved S1 57.2 mm to (39.4, 69.8)
- moved S3 57.2 mm to (77.5, 69.8)
- moved S2 57.1 mm to (58.4, 69.8)
Connections:
- removed net MISO: JP2.1, U$1.11
- removed net MOSI: JP2.4, U$1.10
- removed net SCK: JP2.3, U$1.9
- new net MISO/SW17: JP2.1, S17.S1, U$1.11
- new net MOSI/SW16: JP2.4, S16.S1, U$1.10
- new net N$13: R16.2, S13.A
- new net N$14: R20.2, S17.A
- new net N$15: R21.2, S18.A
- new net N$16: R17.2, S14.A
- new net N$17: R13.2, S10.A
- new net N$18: R9.2, S6.A
- new net N$19: R22.2, S19.A
- new net N$20: R18.2, S15.A
- new net N$21: R14.2, S11.A
- new net N$22: R10.2, S7.A
- new net N$23: R23.2, S20.A
- new net N$24: R19.2, S16.A
- new net N$25: R15.2, S12.A
- new net N$26: R11.2, S8.A
- new net N$4: R8.2, S5.A
- new net N$7: R12.2, S9.A
- new net SCK/SW15: JP2.3, S15.S1, U$1.9
- new net SW10: S10.S1, U$1.30
- new net SW11: S11.S1, U$1.12
- new net SW12: S12.S1, U$1.26
- new net SW13: S13.S1, U$1.32
- new net SW14: S14.S1, U$1.8
- new net SW18: S18.S1, U$1.36
- new net SW19: S19.S1, U$1.37
- new net SW20: S20.S1, U$1.38
- new net SW5: S5.S1, U$1.31
- new net SW6: S6.S1, U$1.27
- new net SW7: S7.S1, U$1.1
- new net SW8: S8.S1, U$1.28
- new net SW9: S9.S1, U$1.29
- net BL: now also R10.1, R11.1, R12.1, R13.1, R14.1, R15.1, R16.1, R17.1, R18.1, R19.1, R20.1, R21.1, R22.1, R23.1, R8.1, R9.1
- net BL_CTRL: now also U$1.18; no longer U$1.27
- net GND: now also S10.K, S10.S2, S11.K, S11.S2, S12.K, S12.S2, S13.K, S13.S2, S14.K, S14.S2, S15.K, S15.S2, S16.K, S16.S2, S17.K, S17.S2, S18.K, S18.S2, S19.K, S19.S2, S20.K, S20.S2, S5.K, S5.S2, S6.K, S6.S2, S7.K, S7.S2, S8.K, S8.S2, S9.K, S9.S2
- net SW1: now also U$1.20; no longer U$1.29
- net SW2: now also U$1.21; no longer U$1.30
- net SW3: now also U$1.19; no longer U$1.31
- net SW4: now also U$1.25; no longer U$1.32
Routing:
- net 5V: track 83.0 -> 0.00 mm, vias 2 -> 0
- net SW4: track 77.4 -> 0.00 mm
- net BL: track 70.5 -> 0.00 mm
- net SW3: track 56.6 -> 0.00 mm
- net SW2: track 35.8 -> 0.00 mm
- net RST: track 18.5 -> 0.00 mm, vias 1 -> 0
- net BL_CTRL: track 12.1 -> 0.00 mm
- net MOSI: track 11.2 -> 0.00 mm
- net SCK: track 9.67 -> 0.00 mm
- net N$8: track 9.48 -> 0.00 mm
- net SW1: track 8.89 -> 0.00 mm
- net N$6: track 6.33 -> 0.00 mm
- net MISO: track 6.29 -> 0.00 mm
- net N$9: track 5.96 -> 0.00 mm
- net N$12: track 5.96 -> 0.00 mm
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- removed copper zone on layer 1, net GND
- removed copper zone on layer 16, net GND
Other:
- board outline removed
- board text removed: "By: Dan Watson 6/4/16 Rev B syncchannel.blogspot.com"
- board text removed: "Cherry MX Keypad"
- board text removed: "SW1"
- board text removed: "SW2"
- board text removed: "SW3"
- board text removed: "SW4"
